Commit message: feat: add ros2_control trajectory controllers and MoveIt integration for UR10e arms

File: src/birobot_description/urdf/birobot.urdf.xacro (robot description, xacro)
@@ -68,4 +68,7 @@
     </collision>
   </link>
+  <!-- Initial home positions property for UR10e arms -->
+  <xacro:property name="initial_positions_file" value="$(find ur_description)/config/initial_positions.yaml"/>
+  <xacro:property name="initial_positions_dict" value="${xacro.load_yaml(initial_positions_file)}"/>
   <!-- Arm 1 instantiation -->
   <xacro:ur_robot
@@ -74,4 +77,6 @@
     parent="workcell_base_link"
     ur_type="ur10e"
+    use_fake_hardware="true"
+    initial_positions="${initial_positions_dict}"
     joint_limits_parameters_file="$(find birobot_description)/vendor/ur_description/config/ur10e/joint_limits.yaml"
     kinematics_parameters_file="$(find birobot_description)/vendor/ur_description/config/ur10e/default_kinematics.yaml"
@@ -86,4 +91,6 @@
     parent="workcell_base_link"
     ur_type="ur10e"
+    use_fake_hardware="true"
+    initial_positions="${initial_positions_dict}"
     joint_limits_parameters_file="$(find birobot_description)/vendor/ur_description/config/ur10e/joint_limits.yaml"
     kinematics_parameters_file="$(find birobot_description)/vendor/ur_description/config/ur10e/default_kinematics.yaml"

File: src/birobot_description/urdf/sensors/depth_camera.urdf.xacro (robot description, xacro)
@@ -76,4 +76,4 @@
       </sensor>
     </gazebo>
-  </xacMacro>
+  </xacro:macro>
 </robot>

Commit message: refactor: unify ros2_control configuration by merging URDF and controller parameters into a single temporary file to resolve controller manager parsing issues.

File: src/birobot_description/urdf/birobot.urdf.xacro (robot description, xacro)
@@ -19,4 +19,10 @@
   <xacro:arg name="table_width" default="0.800"/>
   <xacro:arg name="table_height" default="0.050"/>
+  <xacro:arg name="use_fake_hardware" default="true"/>
+  <xacro:arg name="sim_gazebo" default="false"/>
+  <xacro:arg name="sim_ignition" default="false"/>
+  <xacro:property name="use_fake_hardware" value="$(arg use_fake_hardware)"/>
+  <xacro:property name="sim_gazebo" value="$(arg sim_gazebo)"/>
+  <xacro:property name="sim_ignition" value="$(arg sim_ignition)"/>
   <!-- Convert args to properties for evaluation -->
   <xacro:property name="arm1_x" value="$(arg arm1_x)"/>
@@ -68,6 +74,6 @@
     </collision>
   </link>
-  <!-- Initial home positions property for UR10e arms -->
-  <xacro:property name="initial_positions_file" value="$(find ur_description)/config/initial_positions.yaml"/>
+  <!-- Initial home positions — load from vendored ur_description (shoulder_lift=-1.57, wrist_1=-1.57) -->
+  <xacro:property name="initial_positions_file" value="$(find birobot_description)/vendor/ur_description/config/initial_positions.yaml"/>
   <xacro:property name="initial_positions_dict" value="${xacro.load_yaml(initial_positions_file)}"/>
   <!-- Arm 1 instantiation -->
@@ -77,5 +83,7 @@
     parent="workcell_base_link"
     ur_type="ur10e"
-    use_fake_hardware="true"
+    use_fake_hardware="${use_fake_hardware}"
+    sim_gazebo="${sim_gazebo}"
+    sim_ignition="${sim_ignition}"
     initial_positions="${initial_positions_dict}"
     joint_limits_parameters_file="$(find birobot_description)/vendor/ur_description/config/ur10e/joint_limits.yaml"
@@ -91,5 +99,7 @@
     parent="workcell_base_link"
     ur_type="ur10e"
-    use_fake_hardware="true"
+    use_fake_hardware="${use_fake_hardware}"
+    sim_gazebo="${sim_gazebo}"
+    sim_ignition="${sim_ignition}"
     initial_positions="${initial_positions_dict}"
     joint_limits_parameters_file="$(find birobot_description)/vendor/ur_description/config/ur10e/joint_limits.yaml"
@@ -105,3 +115,13 @@
     <origin xyz="0.0 0.0 1.200" rpy="0.0 1.57079632679 0.0"/>
   </xacro:depth_camera>
+  <!-- Gazebo Sim plugin for ros2_control -->
+  <xacro:if value="${sim_gazebo or sim_ignition}">
+    <xacro:property name="controllers_yaml_path" value="$(find birobot_description)/config/controllers.yaml"/>
+    <gazebo>
+      <plugin filename="gz_ros2_control-system" name="gz_ros2_control::GazeboSimROS2ControlPlugin">
+        <parameters>${controllers_yaml_path}</parameters>
+        <controller_manager_name>controller_manager</controller_manager_name>
+      </plugin>
+    </gazebo>
+  </xacro:if>
 </robot>

File: src/birobot_description/vendor/ur_description/urdf/ur.ros2_control.xacro (robot description, xacro)
@@ -27,10 +27,10 @@
       <hardware>
         <xacro:if value="${sim_gazebo}">
-          <plugin>gazebo_ros2_control/GazeboSystem</plugin>
+          <plugin>gz_ros2_control/GazeboSimSystem</plugin>
         </xacro:if>
         <xacro:if value="${sim_ignition}">
-          <plugin>ign_ros2_control/IgnitionSystem</plugin>
+          <plugin>gz_ros2_control/GazeboSimSystem</plugin>
         </xacro:if>
-        <xacro:if value="${use_fake_hardware}">
+        <xacro:if value="${use_fake_hardware and not (sim_gazebo or sim_ignition)}">
           <plugin>mock_components/GenericSystem</plugin>
           <param name="fake_sensor_commands">${fake_sensor_commands}</param>

Commit message: fix: resolve ROS 2 Jazzy controller manager parameter loading bug by bypassing path-based argument filtering and standardizing use_sim_time settings.

File: src/birobot_description/urdf/birobot.urdf.xacro (robot description, xacro)
@@ -115,11 +115,16 @@
     <origin xyz="0.0 0.0 1.200" rpy="0.0 1.57079632679 0.0"/>
   </xacro:depth_camera>
-  <!-- Gazebo Sim plugin for ros2_control -->
+  <!-- gz_ros2_control plugin. Use only 'parameters' tag - no ros/argument tags. -->
   <xacro:if value="${sim_gazebo or sim_ignition}">
-    <xacro:property name="controllers_yaml_path" value="$(find birobot_description)/config/controllers.yaml"/>
+    <xacro:arg name="controllers_yaml" default="$(find birobot_description)/config/controllers.yaml"/>
+    <xacro:property name="controllers_yaml_path" value="$(arg controllers_yaml)"/>
     <gazebo>
       <plugin filename="gz_ros2_control-system" name="gz_ros2_control::GazeboSimROS2ControlPlugin">
         <parameters>${controllers_yaml_path}</parameters>
         <controller_manager_name>controller_manager</controller_manager_name>
+        <ros>
+          <argument>--params-file</argument>
+          <argument>${controllers_yaml_path}</argument>
+        </ros>
       </plugin>
     </gazebo>

File: src/birobot_description/urdf/sensors/depth_camera.urdf.xacro (robot description, xacro)
@@ -60,18 +60,4 @@
           </noise>
         </camera>
-        <plugin name="${name}_driver" filename="libgazebo_ros_camera.so">
-          <ros>
-            <namespace>/birobot</namespace>
-            <remapping>depth_camera/image_raw:=depth_camera/image_raw</remapping>
-            <remapping>depth_camera/image_depth:=depth_camera/depth_image</remapping>
-            <remapping>depth_camera/camera_info:=depth_camera/camera_info</remapping>
-            <remapping>depth_camera/points:=depth_camera/points</remapping>
-          </ros>
-          <camera_name>depth_camera</camera_name>
-          <frame_name>${name}_optical_frame</frame_name>
-          <hack_baseline>0.07</hack_baseline>
-          <min_depth>0.1</min_depth>
-          <max_depth>5.0</max_depth>
-        </plugin>
       </sensor>
     </gazebo>

Commit message: refactor: standardize all robot joint positions to zero and remove the redundant static joint_state_publisher

File: src/birobot_description/urdf/birobot.urdf.xacro (robot description, xacro)
@@ -74,7 +74,6 @@
     </collision>
   </link>
-  <!-- Initial home positions — load from vendored ur_description (shoulder_lift=-1.57, wrist_1=-1.57) -->
-  <xacro:property name="initial_positions_file" value="$(find birobot_description)/vendor/ur_description/config/initial_positions.yaml"/>
-  <xacro:property name="initial_positions_dict" value="${xacro.load_yaml(initial_positions_file)}"/>
+  <!-- Initial positions: Override vendor defaults and spawn completely flat (0.0) -->
+  <xacro:property name="all_zeros_dict" value="${dict(shoulder_pan_joint=0.0,shoulder_lift_joint=0.0,elbow_joint=0.0,wrist_1_joint=0.0,wrist_2_joint=0.0,wrist_3_joint=0.0)}"/>
   <!-- Arm 1 instantiation -->
   <xacro:ur_robot
@@ -86,5 +85,5 @@
     sim_gazebo="${sim_gazebo}"
     sim_ignition="${sim_ignition}"
-    initial_positions="${initial_positions_dict}"
+    initial_positions="${all_zeros_dict}"
     joint_limits_parameters_file="$(find birobot_description)/vendor/ur_description/config/ur10e/joint_limits.yaml"
     kinematics_parameters_file="$(find birobot_description)/vendor/ur_description/config/ur10e/default_kinematics.yaml"
@@ -102,5 +101,5 @@
     sim_gazebo="${sim_gazebo}"
     sim_ignition="${sim_ignition}"
-    initial_positions="${initial_positions_dict}"
+    initial_positions="${all_zeros_dict}"
     joint_limits_parameters_file="$(find birobot_description)/vendor/ur_description/config/ur10e/joint_limits.yaml"
     kinematics_parameters_file="$(find birobot_description)/vendor/ur_description/config/ur10e/default_kinematics.yaml"

Commit message: feat: update default robot arm home positions to -1.57 rad and integrate configuration from YAML files

File: src/birobot_description/urdf/birobot.urdf.xacro (robot description, xacro)
@@ -74,6 +74,7 @@
     </collision>
   </link>
-  <!-- Initial positions: Override vendor defaults and spawn completely flat (0.0) -->
-  <xacro:property name="all_zeros_dict" value="${dict(shoulder_pan_joint=0.0,shoulder_lift_joint=0.0,elbow_joint=0.0,wrist_1_joint=0.0,wrist_2_joint=0.0,wrist_3_joint=0.0)}"/>
+  <!-- Initial home positions — load from vendored ur_description (shoulder_lift=-1.57, wrist_1=-1.57) -->
+  <xacro:property name="initial_positions_file" value="$(find birobot_description)/vendor/ur_description/config/initial_positions.yaml"/>
+  <xacro:property name="initial_positions_dict" value="${xacro.load_yaml(initial_positions_file)}"/>
   <!-- Arm 1 instantiation -->
   <xacro:ur_robot
@@ -85,5 +86,5 @@
     sim_gazebo="${sim_gazebo}"
     sim_ignition="${sim_ignition}"
-    initial_positions="${all_zeros_dict}"
+    initial_positions="${initial_positions_dict}"
     joint_limits_parameters_file="$(find birobot_description)/vendor/ur_description/config/ur10e/joint_limits.yaml"
     kinematics_parameters_file="$(find birobot_description)/vendor/ur_description/config/ur10e/default_kinematics.yaml"
@@ -101,5 +102,5 @@
     sim_gazebo="${sim_gazebo}"
     sim_ignition="${sim_ignition}"
-    initial_positions="${all_zeros_dict}"
+    initial_positions="${initial_positions_dict}"
     joint_limits_parameters_file="$(find birobot_description)/vendor/ur_description/config/ur10e/joint_limits.yaml"
     kinematics_parameters_file="$(find birobot_description)/vendor/ur_description/config/ur10e/default_kinematics.yaml"

Commit message: refactor: sequence move_group initialization with arm controllers and adjust depth camera mount height

File: src/birobot_description/urdf/birobot.urdf.xacro (robot description, xacro)
@@ -113,5 +113,5 @@
   <!-- Instantiate 3D Depth Camera looking down at table pick zone -->
   <xacro:depth_camera name="depth_camera" parent="workcell_base_link">
-    <origin xyz="0.0 0.0 1.200" rpy="0.0 1.57079632679 0.0"/>
+    <origin xyz="0.0 0.0 2.500" rpy="0.0 1.57079632679 0.0"/>
   </xacro:depth_camera>
   <!-- gz_ros2_control plugin. Use only 'parameters' tag - no ros/argument tags. -->

Commit message: feat: integrate dual-arm 2-finger grippers into simulation and MoveIt planning configurations

File: src/birobot_description/urdf/birobot.urdf.xacro (robot description, xacro)
@@ -109,4 +109,14 @@
     <origin xyz="${arm2_x} ${arm2_y} ${arm2_z}" rpy="${arm2_roll} ${arm2_pitch} ${arm2_yaw}"/>
   </xacro:ur_robot>
+  <!-- Include 2-Finger Gripper macro -->
+  <xacro:include filename="$(find birobot_description)/urdf/grippers/2f_gripper.urdf.xacro"/>
+  <!-- Instantiate 2-Finger Gripper for Arm 1 -->
+  <xacro:two_finger_gripper name="arm1_gripper" prefix="arm1_gripper_" parent="arm1_tool0">
+    <origin xyz="0 0 0" rpy="0 0 0"/>
+  </xacro:two_finger_gripper>
+  <!-- Instantiate 2-Finger Gripper for Arm 2 -->
+  <xacro:two_finger_gripper name="arm2_gripper" prefix="arm2_gripper_" parent="arm2_tool0">
+    <origin xyz="0 0 0" rpy="0 0 0"/>
+  </xacro:two_finger_gripper>
   <!-- Include 3D Depth Camera macro -->
   <xacro:include filename="$(find birobot_description)/urdf/sensors/depth_camera.urdf.xacro"/>

Commit message: feat: update Arm 1 workspace bounds, object spawn positions, camera placement, and grasp orientations

File: src/birobot_description/urdf/birobot.urdf.xacro (robot description, xacro)
@@ -121,7 +121,7 @@
   <!-- Include 3D Depth Camera macro -->
   <xacro:include filename="$(find birobot_description)/urdf/sensors/depth_camera.urdf.xacro"/>
-  <!-- Instantiate 3D Depth Camera looking down at table pick zone -->
+  <!-- Instantiate 3D Depth Camera looking down at Arm 1 table pick zone -->
   <xacro:depth_camera name="depth_camera" parent="workcell_base_link">
-    <origin xyz="0.0 0.0 2.500" rpy="0.0 1.57079632679 0.0"/>
+    <origin xyz="-0.350 0.0 2.500" rpy="0.0 1.57079632679 0.0"/>
   </xacro:depth_camera>
   <!-- gz_ros2_control plugin. Use only 'parameters' tag - no ros/argument tags. -->

Commit message: feat: update perception workspace, depth camera placement, and multi-plane segmentation to target other side of arm

File: src/birobot_description/urdf/birobot.urdf.xacro (robot description, xacro)
@@ -121,7 +121,7 @@
   <!-- Include 3D Depth Camera macro -->
   <xacro:include filename="$(find birobot_description)/urdf/sensors/depth_camera.urdf.xacro"/>
-  <!-- Instantiate 3D Depth Camera looking down at Arm 1 table pick zone -->
+  <!-- Instantiate 3D Depth Camera looking down at Arm 1 pick zone on the other side of Arm 1 -->
   <xacro:depth_camera name="depth_camera" parent="workcell_base_link">
-    <origin xyz="-0.350 0.0 2.500" rpy="0.0 1.57079632679 0.0"/>
+    <origin xyz="-0.850 0.0 2.200" rpy="0.0 1.57079632679 0.0"/>
   </xacro:depth_camera>
   <!-- gz_ros2_control plugin. Use only 'parameters' tag - no ros/argument tags. -->
